File: prueba1.kicad_pcb (KiCad board)
At the start: 2 copper layers, 9 parts, among them J1 GY_63, J2 BMI_270, J3 CMPS2, J4 STH21, J5 ATGM336H, J6 KG200Z, J7 Cargador, U1 RASPBERRY_PI_ZERO_2_W, U2 DC-DC_STEP_UP

Commit message: Nuevos cambios
Parts:
- removed J6: KG200Z, Connector_PinHeader_2.54mm:PinHeader_2x06_P2.54mm_Vertical
- added D1: LED, LED_THT:LED_D5.0mm, F.Cu at (54.5, 107.5)
- added D2: LED, LED_THT:LED_D5.0mm, F.Cu at (62.0, 107.5)
- added J8: KG200Z, madeinhome:kg200z, F.Cu at (42.0, 131.0)
- added J9: BATERIA, Connector_PinHeader_2.54mm:PinHeader_1x02_P2.54mm_Vertical, F.Cu at (42.5, 103.5)
- added Q1: MCP1702-3302E_TO, raspberry:TO127P254X533-3, F.Cu at (77.0, 83.5)
- added R1: 100k, Resistor_THT:R_Axial_DIN0207_L6.3mm_D2.5mm_P10.16mm_Horizontal, F.Cu at (49.0, 112.9)
- added R2: 220K, Resistor_THT:R_Axial_DIN0207_L6.3mm_D2.5mm_P10.16mm_Horizontal, F.Cu at (42.5, 113.1)
- added R3: 4,7k, Resistor_THT:R_Axial_DIN0207_L6.3mm_D2.5mm_P10.16mm_Horizontal, F.Cu at (70.0, 123.0)
- added R4: 4,7k, Resistor_THT:R_Axial_DIN0207_L6.3mm_D2.5mm_P10.16mm_Horizontal, F.Cu at (75.5, 123.0)
- added R5: 2,2k, Resistor_THT:R_Axial_DIN0207_L6.3mm_D2.5mm_P10.16mm_Horizontal, F.Cu at (81.0, 113.0)
- added R6: 220, Resistor_THT:R_Axial_DIN0207_L6.3mm_D2.5mm_P10.16mm_Horizontal, F.Cu at (63.0, 112.9)
- added R7: 220, Resistor_THT:R_Axial_DIN0207_L6.3mm_D2.5mm_P10.16mm_Horizontal, F.Cu at (56.0, 112.9)
- J4: value STH21 -> SHT21
- U1: value RASPBERRY_PI_ZERO_2_W -> TEMP_BAT; footprint raspberry:MODULE_RASPBERRY_PI_ZERO_2_W -> raspberry:TO-92-AMMO
- moved J3 88.7 mm to (84.0, 132.1)
- moved U2 77.6 mm to (88.0, 88.0), turned to 90 degrees
- moved U1 72.0 mm to (37.5, 111.0)
- moved J7 50.8 mm to (41.5, 98.7)
- moved J1 43.7 mm to (101.5, 85.3)
- moved J2 36.8 mm to (111.0, 73.0), turned to -90 degrees
- moved J4 33.3 mm to (101.5, 72.4)
- moved J5 23.6 mm to (126.0, 120.0), turned to -90 degrees
Connections:
- J2 pad 4: /SDO -> /GND
- J2 pad 7: /CSB -> /VCC
- J5 pad 8: unconnected-(J5-Pin_8-Pad8) -> /RX
- J7 pad 10: unconnected-(J7-Pin_10-Pad10) -> /LIPO
- J7 pad 11: unconnected-(J7-Pin_11-Pad11) -> /GND
- J7 pad 8: unconnected-(J7-Pin_8-Pad8) -> /OUT
- U1 pad 1: unconnected-(U1-3V3_1-Pad1) -> /GND
- U1 pad 2: unconnected-(U1-5V_2-Pad2) -> /DQ
- U1 pad 3: unconnected-(U1-GPIO2/SDA1-Pad3) -> /VCC
- U2 pad VIN_N: unconnected-(U2-VIN--PadVIN_N) -> /GND
- U2 pad VIN_P: unconnected-(U2-VIN+-PadVIN_P) -> /OUT
- U2 pad VOUT_N: unconnected-(U2-VOUT--PadVOUT_N) -> /GND
- U2 pad VOUT_P: unconnected-(U2-VOUT+-PadVOUT_P) -> /5V
Routing:
- net /VCC: track 0.00 -> 281.4 mm
- net /SCL: track 0.00 -> 147.0 mm
- net /SDA: track 0.00 -> 145.8 mm
- net /DQ: track 0.00 -> 96.8 mm
- net /GND: track 0.00 -> 93.6 mm
- net /5V: track 0.00 -> 73.2 mm
- net /RX: track 0.00 -> 65.1 mm
- net /OUT: track 0.00 -> 57.9 mm
- net /LIPO: track 0.00 -> 39.0 mm
- net /LED_TX: track 0.00 -> 17.7 mm
- net /ADC: track 0.00 -> 12.7 mm
- net /LED_RX: track 0.00 -> 7.02 mm
- net Net-(D2-A): track 0.00 -> 6.04 mm
- net Net-(D1-A): track 0.00 -> 5.83 mm
- added copper zone on B.Cu, net /GND
Other:
- board outline added: 98.5 x 97 mm
- board text added: "5V"
- board text added: "ADC"
- board text added: "DQ"
- board text added: "D_R"
- board text added: "GND"
- board text added: "LIPO"
- board text added: "MISO"
- board text added: "MOSI"
- board text added: "NC"
- board text added: "OUT"
- board text added: "RX"
- board text added: "RXL"
- board text added: "SCK"
- board text added: "SCL"
- board text added: "SDA"
- board text added: "TXL"
- board text added: "VCC"
- board text added: "VIN"
- board text added: "VOUT"

Commit message: pcb terminada
Parts:
- removed J8: KG200Z, madeinhome:kg200z
- added J10: Conn_01x08_Pin, Connector_PinHeader_2.54mm:PinHeader_1x08_P2.54mm_Vertical, F.Cu at (146.3, 125.5)
- added J11: Conn_01x08_Pin, Connector_PinHeader_2.54mm:PinHeader_1x08_P2.54mm_Vertical, F.Cu at (159.6, 125.3)
- added J6: KG200Z, pines:socket_cont, F.Cu at (67.9, 102.5)
- added REF**: MountingHole_3.2mm_Pad, MountingHole:MountingHole_3.2mm_M3_DIN965_Pad, F.Cu at (71.3, 149.0)
- added REF**: MountingHole_3.2mm_Pad, MountingHole:MountingHole_3.2mm_M3_DIN965_Pad, F.Cu at (166.8, 149.0)
- added REF**: MountingHole_3.2mm_Pad, MountingHole:MountingHole_3.2mm_M3_DIN965_Pad, F.Cu at (166.8, 35.0)
- added REF**: MountingHole_3.2mm_Pad, MountingHole:MountingHole_3.2mm_M3_DIN965_Pad, F.Cu at (71.3, 35.0)
- moved J5 52.6 mm to (163.8, 83.5)
- moved U1 50.7 mm to (71.6, 73.5)
- moved Q1 49.9 mm to (111.1, 47.0)
- moved D1 49.9 mm to (88.5, 71.0)
- moved D2 49.9 mm to (96.0, 71.0)
- moved J1 49.9 mm to (135.6, 48.8)
- moved J2 49.9 mm to (145.1, 36.5)
- moved J3 49.9 mm to (118.1, 95.6)
- moved J4 49.9 mm to (135.6, 35.9)
- moved J7 49.9 mm to (75.6, 62.2)
- moved J9 49.9 mm to (76.6, 67.0)
- moved U2 49.9 mm to (122.1, 51.5)
- moved R2 48.6 mm to (74.6, 76.5)
- moved R1 47.9 mm to (80.1, 76.4)
- moved R3 47.3 mm to (100.1, 86.5)
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Routing:
- net /VDD_3V3: track 0.00 -> 147.1 mm
- net /5V: track 73.2 -> 175.8 mm
- net /D_R: track 0.00 -> 99.3 mm
- net /MOSI: track 0.00 -> 88.2 mm
- net /MISO: track 0.00 -> 86.5 mm
- net /CALEF: track 0.00 -> 83.2 mm
- net /SCK: track 0.00 -> 83.1 mm
- net /CS: track 0.00 -> 80.1 mm
- net /GND: track 93.6 -> 148.5 mm
- net /ADC: track 12.7 -> 63.7 mm
- net /TDI: track 0.00 -> 50.9 mm
- net /SWDIO: track 0.00 -> 48.1 mm
- net /DQ: track 96.8 -> 141.4 mm
- net /SWCLK: track 0.00 -> 44.5 mm
- net /TDO: track 0.00 -> 38.2 mm
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Other:
- board size 98.5 x 97 mm -> 103.8 x 122 mm
- board text added: "3V3"
- board text added: "CALEF"
- board text added: "CS"
- board text added: "LRX"
- board text added: "LTX"
- board text added: "NSS"
- board text added: "PB13"
- board text added: "RESET"
- board text added: "SWCLK"
- board text added: "SWDIO"
- board text added: "TDI"
- board text added: "TDO"
- board text added: "TX"
- board text removed: "NC"
- board text removed: "RXL"
- board text removed: "TXL"
