File: prueba1.kicad_sch (KiCad schematic)
At the start: 9 parts, among them J1 GY_63, J2 BMI_270, J3 CMPS2, J4 STH21, J5 ATGM336H, J6 KG200Z, J7 Cargador, U1 RASPBERRY_PI_ZERO_2_W, U2 DC-DC_STEP_UP

Commit message: Nuevos cambios
Parts:
- removed J6: KG200Z, Connector_PinHeader_2.54mm:PinHeader_2x06_P2.54mm_Vertical, symbol Connector_Generic:Conn_02x06_Counter_Clockwise
- removed U1: RASPBERRY_PI_ZERO_2_W, raspberry:MODULE_RASPBERRY_PI_ZERO_2_W, symbol RASPBERRY_PI_ZERO_2_W:RASPBERRY_PI_ZERO_2_W
- added D1, D2: LED, LED_THT:LED_D5.0mm, symbol Device:LED
- added J8: KG200Z, madeinhome:kg200z, symbol Connector_Generic:Conn_02x08_Counter_Clockwise
- added J9: BATERIA, Connector_PinHeader_2.54mm:PinHeader_1x02_P2.54mm_Vertical, symbol Connector_Generic:Conn_01x02
- added Q1: MCP1702-3302E_TO, raspberry:TO127P254X533-3, symbol MCP1702-3302E_TO:MCP1702-3302E_TO
- added R1: 100k, Resistor_THT:R_Axial_DIN0207_L6.3mm_D2.5mm_P10.16mm_Horizontal, symbol Device:R
- added R2: 220K, Resistor_THT:R_Axial_DIN0207_L6.3mm_D2.5mm_P10.16mm_Horizontal, symbol Device:R
- added R3, R4: 4,7k, Resistor_THT:R_Axial_DIN0207_L6.3mm_D2.5mm_P10.16mm_Horizontal, symbol Device:R
- added R5: 2,2k, Resistor_THT:R_Axial_DIN0207_L6.3mm_D2.5mm_P10.16mm_Horizontal, symbol Device:R
- added R6, R7: 220, Resistor_THT:R_Axial_DIN0207_L6.3mm_D2.5mm_P10.16mm_Horizontal, symbol Device:R
- added U1: TEMP_BAT, raspberry:TO-92-AMMO, symbol DS18B20:DS18B20
- J4: value STH21 -> SHT21
Connections:
- net CSB is gone; now on net VCC: J2.7 (Pin_7)
- net SDO is gone; now on net GND: J2.4 (Pin_4)
- net DATA_READY: now also J8.8 (Pin_8)
- net GND: now also J7.11 (Pin_11), U2.VIN_N (VIN-), U2.VOUT_N (VOUT-), D1.1 (K), D2.1 (K), J8.2 (Pin_2), J9.2 (Pin_2), Q1.1 (GND), R2.1, U1.1 (GND)
- net MISO: now also J8.6 (Pin_6)
- net MOSI: now also J8.5 (Pin_5)
- net RX: now also J5.8 (Pin_8), J8.9 (Pin_9)
- net SCK: now also J8.7 (Pin_7)
- net SCL: now also J8.3 (Pin_3), R3.2
- net SDA: now also J8.4 (Pin_4), R4.2
- net VCC: now also Q1.3 (VOUT), R3.1, R4.1, R5.2, U1.3 (VDD)
- net OUT: now reaches U2.VIN_P (VIN+)
- net OUT: now also J7.8 (Pin_8), Q1.2 (VIN)
- net 5V: now reaches U2.VOUT_P (VOUT+)
- net 5V: now also J8.1 (Pin_1)
- net LIPO: now reaches J7.10 (Pin_10)
- net LIPO: now also J9.1 (Pin_1), R1.1
- new net: D2.2 (A), R6.1
- new net: D1.2 (A), R7.1
- new net ADC: J8.15 (Pin_15), R1.2, R2.2
- new net DQ: J8.14 (Pin_14), R5.1, U1.2 (DQ)
- new net LED_RX: J8.12 (Pin_12), R7.2
- new net LED_TX: J8.13 (Pin_13), R6.2
- no-connect marks 23 -> 34
Other:
- note added: "+bat"
- note added: "-bat"
- note added: "1.0"
- note added: "20/06/26"
- note added: "3V3"
- note added: "5v"
- note added: "BOOSTER"
- note added: "CARGADOR"
- note added: "CONECTOR BAT"
- note added: "CONECTOR QUECTEL"
- note added: "GPS ATGM336H"
- note added: "IMU_AC_GYR BMI270"
- note added: "LEDS TX RX"
- note added: "MAGNETOMETRO CMPS2"
- note added: "MAIN_BOARD_HAPS"
- note added: "PA0"
- note added: "PB1"
- note added: "PB2"
- note added: "PB5"
- note added: "PRESIÓN MS5611"
- note added: "REGULADOR 3V3"
- note added: "RESISTENCIAS PULL UP I2C"
- note added: "TEMP BATERIAS DS18B20"
- note added: "TEMP HUM SHT21"
- note added: "out"
- moved on the sheet: J1, J2, J3, J4, J5, J7, U2

Commit message: pcb terminada
Parts:
- removed J8: KG200Z, madeinhome:kg200z, symbol Connector_Generic:Conn_02x08_Counter_Clockwise
- added J10, J11: Conn_01x08_Pin, Connector_PinHeader_2.54mm:PinHeader_1x08_P2.54mm_Vertical, symbol Connector:Conn_01x08_Pin
- added J6: Conn_01x43_Pin, pines:socket_cont, symbol Connector:Conn_01x43_Pin
Connections:
- net 5V: now also J6.1 (Pin_1), J6.2 (Pin_2)
- net ADC: now also J6.5 (Pin_5)
- net DQ: now also J6.13 (Pin_13)
- net GND: now also J10.2 (Pin_2), J11.2 (Pin_2), J6.12 (Pin_12), J6.17 (Pin_17), J6.22 (Pin_22), J6.3 (Pin_3), J6.31 (Pin_31), J6.32 (Pin_32), J6.33 (Pin_33), J6.34 (Pin_34), J6.35 (Pin_35), J6.36 (Pin_36), J6.37 (Pin_37), J6.39 (Pin_39), J6.4 (Pin_4)
- net LED_RX: now also J6.7 (Pin_7)
- net LED_TX: now also J6.6 (Pin_6)
- net MISO: now also J11.5 (Pin_5), J6.10 (Pin_10)
- net MOSI: now also J11.6 (Pin_6), J6.11 (Pin_11)
- net RX: now also J6.16 (Pin_16)
- net SCK: now also J11.4 (Pin_4), J6.9 (Pin_9)
- net SCL: now also J6.18 (Pin_18)
- net SDA: now also J6.19 (Pin_19)
- new net CALEF: J10.8 (Pin_8), J6.20 (Pin_20)
- new net CS: J11.3 (Pin_3), J6.8 (Pin_8)
- new net D_R: J11.7 (Pin_7), J6.14 (Pin_14)
- new net NSS: J11.8 (Pin_8)
- new net PB13: J6.21 (Pin_21)
- new net RESET_N: J10.5 (Pin_5), J6.30 (Pin_30)
- new net SWCLK: J10.4 (Pin_4), J6.27 (Pin_27)
- new net SWDIO: J10.3 (Pin_3), J6.26 (Pin_26)
- new net TDI: J10.7 (Pin_7), J6.25 (Pin_25)
- new net TDO: J10.6 (Pin_6), J6.29 (Pin_29)
- new net TX: J6.15 (Pin_15)
- new net VDD_3V3: J10.1 (Pin_1), J11.1 (Pin_1), J6.23 (Pin_23), J6.38 (Pin_38), J6.43 (Pin_43)
- no-connect marks 34 -> 36
Other:
- note added: "06/07/26"
- note added: "CONECTORES QUECTEL KG200Z"
- note added: "PA1"
- note added: "PA4"
- note added: "PA5"
- note added: "PA6"
- note added: "PA7"
- note added: "PA8"
- note added: "PB10"
- note added: "PB11"
- note added: "PB12"
- note added: "PB13"
- note added: "PB6"
- note added: "PB7"
- note added: "RESISTENCIAS ADC"
- note added: "SHIELD QUECTEL KG200Z"
- note removed: "20/06/26"
- note removed: "CONECTOR QUECTEL"
- note removed: "PB5"
- moved on the sheet: D1, D2, J1, J2, J3, J4, J5, J7, J9, Q1, R1, R2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
